Commit message: base arena added.
randomization and camera to be added

File: rsc/Triangle/triangle red.urdf (robot description, URDF)
Before this commit: robot arrow, 1 links, 0 joints
Links:
- link Untitled: geometry visual mesh filename=Triangle2.stl scale=0.02996 0.02996 0.00394

File: rsc/Triangle/triangle yellow.urdf (robot description, URDF)
Before this commit: robot base plate, 1 links, 0 joints
Links:
- link Untitled: geometry visual mesh filename=Triangle2.stl scale=0.02996 0.02996 0.00394

File: rsc/base plate/base plate black.urdf (robot description, URDF)
Before this commit: robot circle, 1 links, 0 joints
Links:
- link Untitled: geometry visual box size=0.75 0.75 0.01

File: rsc/base plate/base plate blue.urdf (robot description, URDF)
Before this commit: robot square, 1 links, 0 joints
Links:
- link Untitled: geometry visual box size=0.75 0.75 0.01

File: rsc/base plate/base plate cyan.urdf (robot description, URDF)
Before this commit: robot arrow, 1 links, 0 joints
Links:
- link Untitled: geometry visual box size=0.75 0.75 0.01

File: rsc/base plate/base plate green.urdf (robot description, URDF)
Before this commit: robot arrow, 1 links, 0 joints
Links:
- link Untitled: geometry visual box size=0.75 0.75 0.01

File: rsc/base plate/base plate magenta.urdf (robot description, URDF)
Before this commit: robot arrow, 1 links, 0 joints
Links:
- link Untitled: geometry visual box size=0.75 0.75 0.01

File: rsc/base plate/base plate white.urdf (robot description, URDF)
Before this commit: robot triangle, 1 links, 0 joints
Links:
- link Untitled: geometry visual box size=0.75 0.75 0.01

File: rsc/circle/circle red.urdf (robot description, URDF)
Before this commit: robot arrow, 1 links, 0 joints
Links:
- link Untitled: geometry visual cylinder length=0.01 radius=0.25

File: rsc/circle/circle yellow.urdf (robot description, URDF)
Before this commit: robot arrow, 1 links, 0 joints
Links:
- link Untitled: geometry visual cylinder length=0.01 radius=0.25

File: rsc/square/square red.urdf (robot description, URDF)
Before this commit: robot arrow, 1 links, 0 joints
Links:
- link Untitled: geometry visual box size=0.50 0.50 0.01

File: rsc/square/square yellow.urdf (robot description, URDF)
Before this commit: robot arrow, 1 links, 0 joints
Links:
- link Untitled: geometry visual box size=0.50 0.50 0.01
