Commit message: arena size increased

File: rsc/base plate/base plate black.urdf (robot description, URDF)
Before this commit: robot base plate, 1 links, 0 joints
Links:
- link Untitled: geometry visual box size=1 1 0.01

File: rsc/base plate/base plate blue.urdf (robot description, URDF)
Before this commit: robot base plate, 1 links, 0 joints
Links:
- link Untitled: geometry visual box size=1 1 0.01

File: rsc/base plate/base plate cyan.urdf (robot description, URDF)
Before this commit: robot base plate, 1 links, 0 joints
Links:
- link Untitled: geometry visual box size=1 1 0.01

File: rsc/base plate/base plate green.urdf (robot description, URDF)
Before this commit: robot base plate, 1 links, 0 joints
Links:
- link Untitled: geometry visual box size=1 1 0.01

File: rsc/base plate/base plate magenta.urdf (robot description, URDF)
Before this commit: robot base plate, 1 links, 0 joints
Links:
- link Untitled: geometry visual box size=1 1 0.01

File: rsc/base plate/base plate white.urdf (robot description, URDF)
Before this commit: robot base plate, 1 links, 0 joints
Links:
- link Untitled: geometry visual box size=1 1 0.01
