Commit message: size increased

File: rsc/circle/circle red.urdf (robot description, URDF)
Before this commit: robot circle, 1 links, 0 joints
Links:
- link Untitled: geometry visual cylinder length=0.01 radius=0.3

File: rsc/circle/circle yellow.urdf (robot description, URDF)
Before this commit: robot circle, 1 links, 0 joints
Links:
- link Untitled: geometry visual cylinder length=0.01 radius=0.3

File: rsc/square/square red.urdf (robot description, URDF)
Before this commit: robot square, 1 links, 0 joints
Links:
- link Untitled: geometry visual box size=0.60 0.60 0.01

File: rsc/square/square yellow.urdf (robot description, URDF)
Before this commit: robot square, 1 links, 0 joints
Links:
- link Untitled: geometry visual box size=0.60 0.60 0.01
