Commit message: added aruco on top of car

File: rsc/car/car.urdf (robot description, URDF)
Before this commit: robot husky_robot, 11 links, 10 joints
Links:
- added link aruco; visual mesh filename=meshes/Aruco.stl scale=0.008 0.002 0.008
- added link aruco_base; visual box size=0.4 0.4 0.01
Joints:
- added joint b_to_aruco: type fixed, parent aruco_base, child aruco, origin xyz=0 0 0.001 rpy=0 0 0
- added joint base_to_aruco: type fixed, parent base_link, child aruco_base, origin xyz=0 0 0.3 rpy=0 0 0

Commit message: Update car.urdf

File: rsc/car/car.urdf (robot description, URDF)
Before this commit: robot husky_robot, 13 links, 12 joints
Links:
- link aruco_base: geometry visual box size=0.5 0.5 0.01

Commit message: Update car.urdf

File: rsc/car/car.urdf (robot description, URDF)
Before this commit: robot husky_robot, 13 links, 12 joints
Links:
- link aruco_base: geometry visual box size=0.6 0.6 0.01

Commit message: added Inertia

File: rsc/car/car.urdf (robot description, URDF)
Before this commit: robot husky_robot, 13 links, 12 joints
Links:
- link aruco: mass None -> 0.0001
- link aruco_base: mass None -> 0.0001

Commit message: Update car.urdf

File: rsc/car/car.urdf (robot description, URDF)
Before this commit: robot husky_robot, 13 links, 12 joints
Links:
- link aruco: geometry visual mesh filename=meshes/Aruco.stl scale=0.02 0.002 0.02
- link aruco_base: geometry visual box size=1.2 1.2 0.01
Joints:
- joint base_to_aruco: origin xyz=0 0 0.3 rpy=0 0 0 -> xyz=0 -0.1 0.3 rpy=0 0 0

Commit message: Increased the size of Aruco

File: rsc/car/car.urdf (robot description, URDF)
Before this commit: robot husky_robot, 13 links, 12 joints
Links:
- link aruco: geometry visual mesh filename=meshes/Aruco.stl scale=0.015 0.002 0.015
- link aruco_base: geometry visual box size=1 1 0.01
